File: smartwing1.sch (EAGLE design)
At the start: 8 parts, among them IC1 DSPIC33FJ12GP202, IC2 PIC24FJ16GA002, J1 826926-3, J2 826926-3, J3 826926-3, U1 MPL115A2, U2 MPU-6050, U3 SAM-M8Q

Commit message: petit test
Connections:
- new net N$1: U3.3
Changed lines of the file:
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@@
 </busses>
 <nets>
+<net name="N$1" class="0">
+<segment>
+<wire x1="662.94" y1="-78.74" x2="662.94" y2="-17.78" width="0.1524" layer="91"/>
+<wire x1="662.94" y1="-17.78" x2="698.5" y2="-17.78" width="0.1524" layer="91"/>
+<pinref part="U3" gate="A" pin="3"/>
+<wire x1="698.5" y1="-17.78" x2="698.5" y2="-15.24" width="0.1524" layer="91"/>
+</segment>
+</net>
 </nets>
 </sheet>

Commit message: add lib
Parts:
- removed IC1: DSPIC33FJ12GP202, microchip:DSPIC33FJ12GP202
- removed J1, J2, J3: 826926-3, 826926-3:826926-3
- added ESC1, SERVOMOTEUR1, SERVOMOTEUR2: 826926-3, 826926-3:826926-3
Connections:
- new net N$2: ESC1.2
- new net N$3: ESC1.3
- net N$1: now also ESC1.1; no longer U3.3
Other:
- note removed: "Servo"
- note removed: "esc"
- moved on the sheet: IC2, U1, U2, U3
Changed lines of the file:
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@@
 </class>
 </classes>
+<groups>
+<schematic_group name="ESC"/>
+<schematic_group name="SERVO1"/>
+<schematic_group name="SERVO2"/>
+</groups>
 <parts>
-<part name="IC1" library="microchip" library_urn="urn:adsk.eagle:library:294" deviceset="DSPIC33FJ12GP202" device="" package3d_urn="urn:adsk.eagle:package:20818/2"/>
 <part name="FRAME1" library="frames" library_urn="urn:adsk.eagle:library:229" deviceset="FRAME_C_L" device=""/>
 <part name="U1" library="untitled" deviceset="MPL115A2" device=""/>
 <part name="U2" library="MPU6050" deviceset="MPU-6050" device=""/>
 <part name="IC2" library="microchip" library_urn="urn:adsk.eagle:library:294" deviceset="PIC24FJ16GA002" device="" package3d_urn="urn:adsk.eagle:package:20799/2"/>
-<part name="J1" library="826926-3" deviceset="826926-3" device=""/>
-<part name="J2" library="826926-3" deviceset="826926-3" device=""/>
-<part name="J3" library="826926-3" deviceset="826926-3" device=""/>
+<part name="SERVOMOTEUR2" library="826926-3" deviceset="826926-3" device="" value=""/>
+<part name="SERVOMOTEUR1" library="826926-3" deviceset="826926-3" device="" value="">
+<attribute name="SPICEPREFIX" value="J"/>
+</part>
+<part name="ESC1" library="826926-3" deviceset="826926-3" device="" value=""/>
 <part name="U3" library="SAM_M8Q" deviceset="SAM-M8Q" device=""/>
 </parts>
@@
 <sheet>
 <plain>
-<text x="815.34" y="-30.48" size="1.778" layer="91" rot="R90">Servo</text>
-<text x="815.34" y="35.56" size="1.778" layer="91" rot="R90">Servo</text>
-<text x="815.34" y="-91.44" size="1.778" layer="91" rot="R90">esc</text>
 </plain>
 <instances>
-<instance part="IC1" gate="G$1" x="524.51" y="-177.8" smashed="yes">
-<attribute name="NAME" x="519.43" y="-176.53" size="1.778" layer="95"/>
-<attribute name="VALUE" x="519.43" y="-180.34" size="1.778" layer="96"/>
-</instance>
 <instance part="FRAME1" gate="G$1" x="487.68" y="-203.2" smashed="yes"/>
 <instance part="FRAME1" gate="G$2" x="939.8" y="-203.2" smashed="yes">
@@
 <attribute name="DRAWING_NAME" x="957.58" y="-184.15" size="2.54" layer="94"/>
 </instance>
-<instance part="U1" gate="A" x="678.18" y="-88.9" smashed="yes">
-<attribute name="NAME" x="673.5826" y="-68.3768" size="2.0828" layer="95" ratio="10" rot="SR0"/>
-<attribute name="VALUE" x="672.8714" y="-116.0018" size="2.0828" layer="96" ratio="10" rot="SR0"/>
+<instance part="U1" gate="A" x="868.68" y="-22.86" smashed="yes">
+<attribute name="NAME" x="864.0826" y="-2.3368" size="2.0828" layer="95" ratio="10" rot="SR0"/>
+<attribute name="VALUE" x="863.3714" y="-49.9618" size="2.0828" layer="96" ratio="10" rot="SR0"/>
 </instance>
-<instance part="U2" gate="A" x="716.28" y="-78.74" smashed="yes">
-<attribute name="NAME" x="734.4156" y="-69.6214" size="2.0828" layer="95" ratio="6" rot="SR0"/>
-<attribute name="VALUE" x="733.7806" y="-72.1614" size="2.0828" layer="96" ratio="6" rot="SR0"/>
+<instance part="U2" gate="A" x="688.34" y="33.02" smashed="yes">
+<attribute name="NAME" x="706.4756" y="42.1386" size="2.0828" layer="95" ratio="6" rot="SR0"/>
+<attribute name="VALUE" x="705.8406" y="39.5986" size="2.0828" layer="96" ratio="6" rot="SR0"/>
 </instance>
-<instance part="IC2" gate="G$1" x="680.72" y="-137.16" smashed="yes">
-<attribute name="NAME" x="675.64" y="-135.89" size="1.778" layer="95"/>
-<attribute name="VALUE" x="675.64" y="-139.7" size="1.778" layer="96"/>
+<instance part="IC2" gate="G$1" x="797.56" y="30.48" smashed="yes">
+<attribute name="NAME" x="792.48" y="31.75" size="1.778" layer="95"/>
+<attribute name="VALUE" x="792.48" y="27.94" size="1.778" layer="96"/>
 </instance>
-<instance part="J1" gate="G$1" x="812.8" y="-27.94" smashed="yes">
-<attribute name="NAME" x="807.22" y="-22.86" size="1.778" layer="95"/>
-<attribute name="VALUE" x="807.72" y="-35.56" size="1.778" layer="96"/>
+<instance part="SERVOMOTEUR2" gate="G$1" x="858.52" y="25.4" smashed="yes">
+<attribute name="NAME" x="852.94" y="30.48" size="1.778" layer="95"/>
+<attribute name="VALUE" x="853.44" y="17.78" size="1.778" layer="96"/>
 </instance>
-<instance part="J2" gate="G$1" x="812.8" y="38.1" smashed="yes">
-<attribute name="NAME" x="807.22" y="43.18" size="1.778" layer="95"/>
-<attribute name="VALUE" x="807.72" y="30.48" size="1.778" layer="96"/>
+<instance part="SERVOMOTEUR1" gate="G$1" x="858.52" y="45.72" smashed="yes">
+<attribute name="NAME" x="852.94" y="50.8" size="1.778" layer="95"/>
+<attribute name="VALUE" x="853.44" y="38.1" size="1.778" layer="96"/>
 </instance>
-<instance part="J3" gate="G$1" x="812.8" y="-91.44" smashed="yes">
-<attribute name="NAME" x="807.22" y="-86.36" size="1.778" layer="95"/>
-<attribute name="VALUE" x="807.72" y="-99.06" size="1.778" layer="96"/>
+<instance part="ESC1" gate="G$1" x="805.18" y="86.36" smashed="yes" rot="R90">
+<attribute name="NAME" x="800.1" y="80.78" size="1.778" layer="95" rot="R90"/>
+<attribute name="VALUE" x="812.8" y="81.28" size="1.778" layer="96" rot="R90"/>
 </instance>
-<instance part="U3" gate="A" x="695.96" y="-10.16" smashed="yes">
-<attribute name="NAME" x="711.5556" y="-1.0414" size="2.0828" layer="95" ratio="6" rot="SR0"/>
-<attribute name="VALUE" x="710.9206" y="-3.5814" size="2.0828" layer="96" ratio="6" rot="SR0"/>
+<instance part="U3" gate="A" x="774.7" y="-15.24" smashed="yes">
+<attribute name="NAME" x="790.2956" y="-6.1214" size="2.0828" layer="95" ratio="6" rot="SR0"/>
+<attribute name="VALUE" x="789.6606" y="-8.6614" size="2.0828" layer="96" ratio="6" rot="SR0"/>
 </instance>
 </instances>
@@
 <net name="N$1" class="0">
 <segment>
-<wire x1="662.94" y1="-78.74" x2="662.94" y2="-17.78" width="0.1524" layer="91"/>
-<wire x1="662.94" y1="-17.78" x2="698.5" y2="-17.78" width="0.1524" layer="91"/>
-<pinref part="U3" gate="A" pin="3"/>
-<wire x1="698.5" y1="-17.78" x2="698.5" y2="-15.24" width="0.1524" layer="91"/>
+<pinref part="ESC1" gate="G$1" pin="1"/>
+<wire x1="802.64" y1="76.2" x2="802.64" y2="63.5" width="0.1524" layer="91"/>
+</segment>
+</net>
+<net name="N$2" class="0">
+<segment>
+<pinref part="ESC1" gate="G$1" pin="2"/>
+<wire x1="805.18" y1="76.2" x2="805.18" y2="63.5" width="0.1524" layer="91"/>
+</segment>
+</net>
+<net name="N$3" class="0">
+<segment>
+<pinref part="ESC1" gate="G$1" pin="3"/>
+<wire x1="807.72" y1="76.2" x2="807.72" y2="63.5" width="0.1524" layer="91"/>
 </segment>
 </net>
@@
 packages will not be understood (or retained) with this version.
 </note>
+<note version="9.5" severity="warning">
+Since Version 9.5, EAGLE supports persistent groups with
+schematics, and board files. Those persistent groups
+will not be understood (or retained) with this version.
+</note>
 </compatibility>

Commit message: V1
Parts:
- added C1: 100nF, rcl:C-EU075-032X103
- added CHANEL1, CHANEL2, CHANEL3, CHANEL4: 826926-3, 826926-3:826926-3
- added JP1: (no value), pinhead:PINHD-1X5
- added R1: 10K, rcl:R-EU_0204/5
- added R2: 10k, rcl:R-EU_0204/5
- added R3: 100, rcl:R-EU_0204/5
- added SW1: CT10-XXXX-A2, switch-coto:CT10-XXXX-A2
Connections:
- removed net N$1: ESC1.1
- removed net N$2: ESC1.2
- new net 0: CHANEL4.1
- new net GND: C1.1, ESC1.1, R3.1, SERVOMOTEUR1.1, SERVOMOTEUR2.1
- new net N$13: R2.1
- new net N$14: JP1.1
- new net N$5: C1.2, R1.1, R2.2, SW1.1
- new net N$7: R3.2, SW1.2
- new net N$8: IC2.VDD@1
- new net N$9: CHANEL4.2
- new net S: JP1.4, JP1.5
- new net VCC: ESC1.2, R1.2, SERVOMOTEUR1.2, SERVOMOTEUR2.2
Other:
- note added: "V1.0.0"
- moved on the sheet: ESC1, IC2, SERVOMOTEUR1, SERVOMOTEUR2, U1, U2, U3

Commit message: V1.0.01
Parts:
- added C10, C11, C6, C7, C8, C9: 100nF, rcl:C-EU075-032X103
- added C2, C3, C4: 0.1uF, rcl:C-EU050-045X075
- added C5: 10uF, rcl:C-EU050-045X075
- added IC1: PIC24HJ12GP202, Smartwing_LIB_PIC:PIC24HJ12GP202
- IC2: value PIC24FJ16GA002 -> (none); device microchip:PIC24FJ16GA002 -> v-reg:78LXX
Connections:
- removed net N$13: R2.1
- removed net S: JP1.4, JP1.5
- new net MCLR: IC1.!MCLR, JP1.1, R2.1
- new net N$1: C4.1, IC1.VSS@1
- new net N$15: CHANEL2.1
- new net N$16: IC1.OSC1/CLKI/CN30/RA2
- new net N$17: IC1.OSC2/CLKO/CN29/RA3
- new net N$2: IC1.PGED2/AN0/VREF+/CN2/RA0
- new net N$20: C3.1, C4.2, IC1.VDD@1
- new net N$22: C2.1, IC1.VDD@2
- new net N$23: C2.2, IC1.VSS@2
- new net N$26: IC1.AN8/RP13(1)/CN13/RB13
- new net N$27: IC1.AN9/RP12(1)/CN14/RB12
- new net N$28: IC1.TMS/RP11(1)/CN15/RB11
- new net N$29: IC1.TDI/RP10(1)/CN16/RB10
- new net N$3: IC1.PGEC2/AN1/VREF-/CN3/RA1
- new net N$30: C5.1, IC1.VCAP
- new net N$31: C3.2, IC1.VSS
- new net N$32: IC1.TDO/SDA1/RP9(1)/CN21/RB9
- new net N$33: IC1.TCK/SCL1/RP8(1)/CN22/RB8
- new net N$34: IC1.INT0/RP7(1)/CN23/RB7
- new net N$35: IC1.ASCL1/RP6(1)/CN24/RB6
- new net N$37: CHANEL3.2
- new net N$38: CHANEL3.1
- new net N$6: C6.2, C7.1, IC2.GND
- new net PGC: IC1.PGEC1/AN3/RP1(1)/CN5/RB1, JP1.5
- new net PGD: IC1.PGED1/AN2/RP0(1)/CN4/RB0, JP1.4
- new net PIN1: ESC1.3, IC1.AN4/RP2(1)/CN6/RB2
- new net PIN2: IC1.AN5/RP3(1)/CN7/RB3, SERVOMOTEUR1.3
- new net PIN3: IC1.PGED3/SOSC/RP4(1)/CN1/RB4, SERVOMOTEUR2.3
- new net PIN4: CHANEL1.3, IC1.PGEC3/SOSCO/T1CK/CN0/RA4
- new net PIN5: CHANEL2.3, IC1.ASDA1/RP5(1)/CN27/RB5
- new net PIN6: CHANEL3.3, IC1.AN6/RP15(1)/CN11/RB15
- new net PIN7: CHANEL4.3, IC1.AN7/RP14(1)/CN12/RB14
- new net VBAT: C6.1, IC2.IN
- net 0: now also C10.1, C11.2, C8.2, C9.1, ESC1.1, SERVOMOTEUR1.1, SERVOMOTEUR2.1
- net GND: now also C5.2; no longer ESC1.1, SERVOMOTEUR1.1, SERVOMOTEUR2.1
- net N$12: now also CHANEL1.1; no longer ESC1.3
- net N$14: now also CHANEL2.2; no longer JP1.1
- net N$8: now also C7.2, IC2.OUT; no longer IC2.VDD@1
- net N$9: now also CHANEL1.2; no longer CHANEL4.2
- net VCC: now also C10.2, C11.1, C8.1, C9.2, CHANEL4.2
Other:
- note added: "VCC = 3v3"
- moved on the sheet: C1, CHANEL1, CHANEL2, CHANEL3, CHANEL4, ESC1, R1, R2, R3, SERVOMOTEUR1, SERVOMOTEUR2, SW1
