File: smartwing1.sch (EAGLE design)
At the start: 63 parts, among them IC3 PIC24FJ64GB002, SW1 CT10-XXXX-A2, U1 SEN0142, U2 SN74LVC1T45DBVT, U3 SN74LVC1T45DBVT, U4 SN74LVC1T45DBVT, U5 SN74LVC1T45DBVT, U6 SN74LVC1T45DBVT, U7 SN74LVC1T45DBVT, U8 SN74LVC1T45DBVT

Commit message: chgmnt_baro_et_sda_scl_axelle
Parts:
- removed R4, R5: 4.7k, rcl:R-EU_0207/7
Connections:
- removed net MPL_SCL: R5.2, U$1.SCL
- removed net MPL_SDA: R4.2, U$1.SDA
- removed net N$1: U$1.RST
- removed net N$17: U$1.SDWN
- removed net SEN_SCL: IC3.TCK/USBOEN/SCL1/RP8/PMD4/CN22/RB8, U1.SCL
- removed net SEN_SDA: IC3.TDO/SDA1/RP9/PMD3/RCV/CN21/RB9, U1.SDA
- new net SCL: IC3.TCK/USBOEN/SCL1/RP8/PMD4/CN22/RB8, U$1.SCL, U1.SCL
- new net SDA: IC3.TDO/SDA1/RP9/PMD3/RCV/CN21/RB9, U$1.SDA, U1.SDA
- net VCC: no longer R4.1, R5.1
Changed lines of the file:
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@@
 <part name="P+12" library="supply1" library_urn="urn:adsk.eagle:library:371" deviceset="VCC" device=""/>
 <part name="X_16" library="ngspice-simulation" library_urn="urn:adsk.eagle:library:527439" deviceset="GND" device=""/>
-<part name="R4" library="rcl" library_urn="urn:adsk.eagle:library:334" deviceset="R-EU_" device="0207/7" package3d_urn="urn:adsk.eagle:package:23493/2" value="4.7k"/>
-<part name="R5" library="rcl" library_urn="urn:adsk.eagle:library:334" deviceset="R-EU_" device="0207/7" package3d_urn="urn:adsk.eagle:package:23493/2" value="4.7k"/>
-<part name="P+13" library="supply1" library_urn="urn:adsk.eagle:library:371" deviceset="VCC" device=""/>
 <part name="U1" library="MPU6050" deviceset="SEN0142" device=""/>
 <part name="X_18" library="ngspice-simulation" library_urn="urn:adsk.eagle:library:527439" deviceset="GND" device=""/>
@@
 </instance>
 <instance part="X_16" gate="G$1" x="942.34" y="-109.22" smashed="yes" grouprefs="MIKROE"/>
-<instance part="R4" gate="G$1" x="810.26" y="-134.62" smashed="yes" rot="R90" grouprefs="MPL115A2">
-<attribute name="NAME" x="808.7614" y="-138.43" size="1.778" layer="95" rot="R90"/>
-<attribute name="VALUE" x="813.562" y="-138.43" size="1.778" layer="96" rot="R90"/>
-</instance>
-<instance part="R5" gate="G$1" x="817.88" y="-134.62" smashed="yes" rot="R90" grouprefs="MPL115A2">
-<attribute name="NAME" x="816.3814" y="-138.43" size="1.778" layer="95" rot="R90"/>
-<attribute name="VALUE" x="821.182" y="-138.43" size="1.778" layer="96" rot="R90"/>
-</instance>
-<instance part="P+13" gate="VCC" x="815.34" y="-144.78" smashed="yes" rot="R180" grouprefs="MPL115A2">
-<attribute name="VALUE" x="817.88" y="-142.24" size="1.778" layer="96" rot="R270"/>
-</instance>
 <instance part="U1" gate="U2" x="650.24" y="-83.82" smashed="yes" grouprefs="SEN0142">
 <attribute name="NAME" x="668.3756" y="-74.7014" size="2.0828" layer="95" ratio="6" rot="SR0"/>
@@
 <junction x="881.38" y="-99.06" grouprefs="MIKROE"/>
 <pinref part="U$2" gate="G$1" pin="3.3V"/>
-</segment>
-<segment>
-<pinref part="R5" gate="G$1" pin="1"/>
-<wire x1="817.88" y1="-142.24" x2="817.88" y2="-139.7" width="0.1524" layer="91" grouprefs="MPL115A2"/>
-<pinref part="R4" gate="G$1" pin="1"/>
-<wire x1="810.26" y1="-139.7" x2="810.26" y2="-142.24" width="0.1524" layer="91" grouprefs="MPL115A2"/>
-<wire x1="810.26" y1="-142.24" x2="815.34" y2="-142.24" width="0.1524" layer="91" grouprefs="MPL115A2"/>
-<pinref part="P+13" gate="VCC" pin="VCC"/>
-<wire x1="815.34" y1="-142.24" x2="817.88" y2="-142.24" width="0.1524" layer="91" grouprefs="MPL115A2"/>
-<junction x="815.34" y="-142.24" grouprefs="MPL115A2"/>
 </segment>
 </net>
@@
 </segment>
 </net>
-<net name="MPL_SDA" class="0">
+<net name="SDA" class="0">
 <segment>
 <pinref part="U$1" gate="G$1" pin="SDA"/>
 <label x="807.72" y="-116.84" size="1.778" layer="95" rot="R270" grouprefs="MPL115A2"/>
-<wire x1="810.26" y1="-114.3" x2="810.26" y2="-129.54" width="0.1524" layer="91" grouprefs="MPL115A2"/>
-<pinref part="R4" gate="G$1" pin="2"/>
+<wire x1="810.26" y1="-114.3" x2="810.26" y2="-121.92" width="0.1524" layer="91" grouprefs="MPL115A2"/>
+</segment>
+<segment>
+<pinref part="U1" gate="U2" pin="SDA"/>
+<wire x1="693.42" y1="-86.36" x2="701.04" y2="-86.36" width="0.1524" layer="91" grouprefs="SEN0142"/>
+<label x="695.96" y="-86.36" size="1.778" layer="95" grouprefs="SEN0142"/>
+</segment>
+<segment>
+<pinref part="IC3" gate="G$1" pin="TDO/SDA1/RP9/PMD3/RCV/CN21/RB9"/>
+<wire x1="850.9" y1="0" x2="863.6" y2="0" width="0.1524" layer="91"/>
+<label x="858.52" y="0" size="1.778" layer="91"/>
 </segment>
 </net>
@@
 </segment>
 </net>
-<net name="MPL_SCL" class="0">
+<net name="SCL" class="0">
 <segment>
 <pinref part="U$1" gate="G$1" pin="SCL"/>
-<wire x1="817.88" y1="-114.3" x2="817.88" y2="-129.54" width="0.1524" layer="91" grouprefs="MPL115A2"/>
+<wire x1="817.88" y1="-114.3" x2="817.88" y2="-121.92" width="0.1524" layer="91" grouprefs="MPL115A2"/>
 <label x="815.34" y="-116.84" size="1.778" layer="95" rot="R270" grouprefs="MPL115A2"/>
-<pinref part="R5" gate="G$1" pin="2"/>
+</segment>
+<segment>
+<pinref part="U1" gate="U2" pin="SCL"/>
+<wire x1="693.42" y1="-88.9" x2="701.04" y2="-88.9" width="0.1524" layer="91" grouprefs="SEN0142"/>
+<label x="695.96" y="-88.9" size="1.778" layer="95" grouprefs="SEN0142"/>
+</segment>
+<segment>
+<pinref part="IC3" gate="G$1" pin="TCK/USBOEN/SCL1/RP8/PMD4/CN22/RB8"/>
+<wire x1="850.9" y1="-5.08" x2="863.6" y2="-5.08" width="0.1524" layer="91"/>
+<label x="858.52" y="-5.08" size="1.778" layer="95"/>
 </segment>
 </net>
@@
 <wire x1="721.36" y1="40.64" x2="708.66" y2="40.64" width="0.1524" layer="91"/>
 <label x="708.66" y="40.64" size="1.778" layer="95"/>
-</segment>
-</net>
-<net name="N$1" class="0">
-<segment>
-<pinref part="U$1" gate="G$1" pin="RST"/>
-<wire x1="802.64" y1="-114.3" x2="802.64" y2="-142.24" width="0.1524" layer="91" grouprefs="MPL115A2"/>
-</segment>
-</net>
-<net name="SEN_SDA" class="0">
-<segment>
-<pinref part="U1" gate="U2" pin="SDA"/>
-<wire x1="693.42" y1="-86.36" x2="711.2" y2="-86.36" width="0.1524" layer="91" grouprefs="SEN0142"/>
-<label x="711.2" y="-83.82" size="1.778" layer="95" rot="R180" grouprefs="SEN0142"/>
-</segment>
-<segment>
-<pinref part="IC3" gate="G$1" pin="TDO/SDA1/RP9/PMD3/RCV/CN21/RB9"/>
-<wire x1="850.9" y1="0" x2="863.6" y2="0" width="0.1524" layer="91"/>
-<label x="863.6" y="2.54" size="1.778" layer="91" rot="R180"/>
-</segment>
-</net>
-<net name="SEN_SCL" class="0">
-<segment>
-<pinref part="U1" gate="U2" pin="SCL"/>
-<wire x1="693.42" y1="-88.9" x2="711.2" y2="-88.9" width="0.1524" layer="91" grouprefs="SEN0142"/>
-<label x="711.2" y="-86.36" size="1.778" layer="95" rot="R180" grouprefs="SEN0142"/>
-</segment>
-<segment>
-<pinref part="IC3" gate="G$1" pin="TCK/USBOEN/SCL1/RP8/PMD4/CN22/RB8"/>
-<wire x1="850.9" y1="-5.08" x2="863.6" y2="-5.08" width="0.1524" layer="91"/>
-<label x="863.6" y="-2.54" size="1.778" layer="95" rot="R180"/>
 </segment>
 </net>
@@
 </segment>
 </net>
-<net name="N$17" class="0">
-<segment>
-<pinref part="U$1" gate="G$1" pin="SDWN"/>
-<wire x1="795.02" y1="-114.3" x2="795.02" y2="-142.24" width="0.1524" layer="91"/>
-</segment>
-</net>
